File: hardware/hardware.kicad_pcb (KiCad board)
At the start: 2 copper layers, 52 parts, among them J1 120V, J2 USB_B, J3 temp0, J4 temp1, J5 heat0, J6 heat1, SW1 BOOT, SW2 RST, U1 AZ1117CR-3.3, U2 ESP32-C3-MINI-1U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

Commit message: layout WIP
Parts:
- TP1, TP2: footprint TestPoint:TestPoint_Plated_Hole_D2.0mm -> TestPoint:TestPoint_THTPad_D1.0mm_Drill0.5mm
- moved R10 145.7 mm to (147.0, 129.0), turned to -90 degrees
- moved R14 142.0 mm to (128.0, 117.0), turned to 90 degrees
- moved R3 139.3 mm to (142.5, 129.0), turned to -90 degrees
- moved C2 138.2 mm to (131.5, 133.2), turned to 90 degrees
- moved D1 137.5 mm to (132.2, 138.5), turned to 180 degrees
- moved D4 136.5 mm to (145.5, 129.0), turned to 90 degrees
- moved C8 136.3 mm to (153.5, 140.2), turned to -90 degrees
- moved D2 135.1 mm to (123.2, 132.5), turned to -90 degrees
- moved R16 126.3 mm to (135.5, 105.0), turned to -90 degrees
- moved TP1 125.8 mm to (136.8, 137.0)
- moved D5 125.8 mm to (122.5, 73.5), turned to -90 degrees
- moved F1 124.4 mm to (123.2, 137.0), turned to 90 degrees
- moved U1 123.9 mm to (125.8, 126.2), turned to -90 degrees
- moved R5 122.2 mm to (122.5, 76.5), turned to 90 degrees
- moved TP2 121.7 mm to (136.8, 139.5)
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Connections:
- D1 pad 2: /USB_D- -> /USB_D+
- D1 pad 3: /USB_D+ -> /USB_D-
- J1 pad 2: /120V_NEUTRAL -> /120V_HOT
- J1 pad 3: /120V_HOT -> /120V_NEUTRAL
- J5 pad 1: /120V_NEUTRAL -> /heater0/T1
- J5 pad 2: /heater0/T1 -> /120V_NEUTRAL
- U2 pad 12: /SCK -> /MISO
- U2 pad 16: /CS1 -> /SCK
- U2 pad 18: /HEAT0 -> /ZCD
- U2 pad 19: /HEAT1 -> /LED
- U2 pad 20: /LED -> /HEAT1
- U2 pad 21: /ZCD -> /HEAT0
- U2 pad 6: /MISO -> /CS1
Routing:
- net +3V3: track 0.00 -> 86.8 mm, vias 0 -> 7
- net /120V_HOT: track 0.00 -> 65.3 mm
- net +5V: track 0.00 -> 60.2 mm
- net /ZCD: track 0.00 -> 38.1 mm
- net /SCK: track 0.00 -> 30.5 mm
- net /MISO: track 0.00 -> 28.8 mm
- net /HEAT0: track 0.00 -> 27.2 mm, vias 0 -> 2
- net /HEAT1: track 0.00 -> 27.0 mm, vias 0 -> 2
- net /USB_D-: track 0.00 -> 21.0 mm
- net Net-(C3-Pad1): track 0.00 -> 20.6 mm, vias 0 -> 1
- net /120V_NEUTRAL: track 0.00 -> 20.2 mm
- net Net-(R14-Pad2): track 0.00 -> 18.7 mm
- net /CS0: track 0.00 -> 16.1 mm
- net /CS1: track 0.00 -> 14.2 mm
- net /USB_D+: track 0.00 -> 14.1 mm
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- added copper zone on B.Cu, net /120V_NEUTRAL
- added copper zone on F.Cu, net /120V_NEUTRAL
- added copper zone on F.Cu, net /heater0/T1
- added copper zone on F.Cu, net /heater1/T1
- added copper zone on B.Cu, net Earth
- added copper zone on F.Cu, net Earth
- added copper zone on B.Cu, net GND
- added copper zone on F.Cu, net GND
Other:
- board outline added: 60 x 75 mm

Commit message: finished layout
Parts:
- TP1, TP2: footprint TestPoint:TestPoint_THTPad_D1.0mm_Drill0.5mm -> TestPoint:TestPoint_Pad_D2.0mm
- moved D5 0.75 mm to (122.5, 74.2)
- moved R5 0.75 mm to (122.5, 77.2)
- moved R9 0.50 mm to (175.2, 110.8)
- moved TP2 0.50 mm to (136.8, 140.0)
Connections:
- R8 pad 1: /120V_HOT -> /120V_NEUTRAL
- R9 pad 2: /120V_NEUTRAL -> /120V_HOT
Routing:
- net /heater0/T1: track 0.00 -> 46.5 mm, vias 0 -> 1
- net Net-(D6-Pad3): track 2.34 -> 34.5 mm, vias 0 -> 1
- net /heater1/T1: track 0.00 -> 19.5 mm
- net /120V_NEUTRAL: track 20.2 -> 35.4 mm
- net /120V_HOT: track 65.3 -> 58.7 mm, vias 0 -> 1
- net Net-(D7-Pad3): track 8.01 -> 9.52 mm
- net +5V: track 60.2 -> 59.4 mm
- net Net-(TP2-Pad1): track 3.30 -> 3.80 mm
- net GND: vias 0 -> 26
- net Earth: vias 0 -> 120
- added copper zone on F.Cu, net /120V_HOT
- removed copper zone on B.Cu, net /120V_NEUTRAL
Other:
- board text added: "+"
- board text added: "AC input"
- board text added: "BOOT"
- board text added: "G"
- board text added: "L"
- board text added: "N"
- board text added: "OSRO v1 Matt Tran"
- board text added: "RST"
- board text added: "danger! high voltage!"
- board text added: "heater0 heater1"
- board text added: "temp0 temp1"

Commit message: added bang-bang implementation
Parts:
- R11, R14, R4: value 150 -> 100
- R12, R15: value 150 -> 22
- R13, R16: value 150 -> 10k
Changed lines of the file:
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@@
       (effects (font (size 1 1) (thickness 0.15)))
     )
-    (fp_text value "150" (at 0 1.43 90) (layer "F.Fab")
+    (fp_text value "10k" (at 0 1.43 90) (layer "F.Fab")
       (effects (font (size 1 1) (thickness 0.15)))
     )
@@
       (effects (font (size 1 1) (thickness 0.15)))
     )
-    (fp_text value "150" (at 0 1.43 90) (layer "F.Fab")
+    (fp_text value "100" (at 0 1.43 90) (layer "F.Fab")
       (effects (font (size 1 1) (thickness 0.15)))
     )
@@
       (effects (font (size 1 1) (thickness 0.15)))
     )
-    (fp_text value "150" (at 0 1.43 90) (layer "F.Fab")
+    (fp_text value "22" (at 0 1.43 90) (layer "F.Fab")
       (effects (font (size 1 1) (thickness 0.15)))
     )
@@
       (effects (font (size 1 1) (thickness 0.15)))
     )
-    (fp_text value "150" (at 0 1.43 90) (layer "F.Fab")
+    (fp_text value "100" (at 0 1.43 90) (layer "F.Fab")
       (effects (font (size 1 1) (thickness 0.15)))
     )
@@
       (effects (font (size 1 1) (thickness 0.15)))
     )
-    (fp_text value "150" (at 0 1.43 90) (layer "F.Fab")
+    (fp_text value "22" (at 0 1.43 90) (layer "F.Fab")
       (effects (font (size 1 1) (thickness 0.15)))
     )
@@
       (effects (font (size 1 1) (thickness 0.15)))
     )
-    (fp_text value "150" (at 0 1.43 90) (layer "F.Fab")
+    (fp_text value "10k" (at 0 1.43 90) (layer "F.Fab")
       (effects (font (size 1 1) (thickness 0.15)))
     )
@@
       (effects (font (size 1 1) (thickness 0.15)))
     )
-    (fp_text value "150" (at 0 1.43 90) (layer "F.Fab")
-      (effects (font (size 1 1) (thickness 0.15)))
-    )
+    (fp_text value "100" (at 0 1.43 90) (layer "F.Fab")
+      (effects (font (size 1 1) (thickness 0.15)))
+    )
