File: hardware/thermocouple.kicad_sch (KiCad schematic)
At the start: 3 parts

Commit message: assigned footprints
Parts:
- C10: renamed from C?; footprint (none) -> Capacitor_SMD:C_0603_1608Metric
- R7: renamed from R?; footprint (none) -> Resistor_SMD:R_0603_1608Metric
- gave numbers to parts that had none: 1
Changed lines of the file:
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@@
   (symbol (lib_id "power:+3V3") (at 137.16 110.49 180)
     (in_bom yes) (on_board yes)
-    (property "Reference" "#PWR?" (id 0) (at 137.16 106.68 0)
+    (property "Reference" "#PWR029" (id 0) (at 137.16 106.68 0)
       (effects (font (size 1.27 1.27)) hide)
     )
@@
   (symbol (lib_id "Device:R_Small") (at 137.16 107.95 0)
     (in_bom yes) (on_board yes)
-    (property "Reference" "R?" (id 0) (at 138.43 106.68 0)
+    (property "Reference" "R7" (id 0) (at 138.43 106.68 0)
       (effects (font (size 1.27 1.27)) (justify left))
     )
@@
       (effects (font (size 1.27 1.27)) (justify left))
     )
-    (property "Footprint" "" (id 2) (at 137.16 107.95 0)
+    (property "Footprint" "Resistor_SMD:R_0603_1608Metric" (id 2) (at 137.16 107.95 0)
       (effects (font (size 1.27 1.27)) hide)
     )
@@
   (symbol (lib_id "extraparts:MAX6675") (at 148.59 101.6 0)
     (in_bom yes) (on_board yes)
-    (property "Reference" "U?" (id 0) (at 142.24 91.44 0)
+    (property "Reference" "U4" (id 0) (at 142.24 91.44 0)
       (effects (font (size 1.27 1.27)) (justify left))
     )
@@
   (symbol (lib_id "power:GND") (at 148.59 110.49 0)
     (in_bom yes) (on_board yes) (fields_autoplaced)
-    (property "Reference" "#PWR?" (id 0) (at 148.59 116.84 0)
+    (property "Reference" "#PWR031" (id 0) (at 148.59 116.84 0)
       (effects (font (size 1.27 1.27)) hide)
     )
@@
   (symbol (lib_id "Device:C_Small") (at 152.4 86.36 0)
     (in_bom yes) (on_board yes)
-    (property "Reference" "C?" (id 0) (at 154.94 85.09 0)
+    (property "Reference" "C10" (id 0) (at 154.94 85.09 0)
       (effects (font (size 1.27 1.27)) (justify left))
     )
@@
       (effects (font (size 1.27 1.27)) (justify left))
     )
-    (property "Footprint" "" (id 2) (at 152.4 86.36 0)
+    (property "Footprint" "Capacitor_SMD:C_0603_1608Metric" (id 2) (at 152.4 86.36 0)
       (effects (font (size 1.27 1.27)) hide)
     )
@@
   (symbol (lib_id "power:+3V3") (at 148.59 83.82 0)
     (in_bom yes) (on_board yes) (fields_autoplaced)
-    (property "Reference" "#PWR?" (id 0) (at 148.59 87.63 0)
+    (property "Reference" "#PWR030" (id 0) (at 148.59 87.63 0)
       (effects (font (size 1.27 1.27)) hide)
     )
@@
   (symbol (lib_id "power:GND") (at 152.4 88.9 0)
     (in_bom yes) (on_board yes) (fields_autoplaced)
-    (property "Reference" "#PWR?" (id 0) (at 152.4 95.25 0)
+    (property "Reference" "#PWR032" (id 0) (at 152.4 95.25 0)
       (effects (font (size 1.27 1.27)) hide)
     )

Commit message: update to KiCad 7
Parts:
- renumbered C10 to C9, R7 to R6, U4 to U3
